File: TriacSwitch/TriacSwitch.sch (KiCad schematic (older format))
At the start: 10 parts

Commit message: Triac revision
Connections:
- net Load: no longer D?.3 (G), U?.4
- new net: D?.3 (G), U?.4
Changed lines of the file:
@@
 LIBS:contrib
 LIBS:valves
+LIBS:TriacSwitch-cache
 EELAYER 25 0
 EELAYER END
@@
 	3850 2450 3800 2450
 Wire Wire Line
-	3800 2450 3800 2800
-Wire Wire Line
-	3200 2800 5400 2800
-Connection ~ 4000 2800
-Connection ~ 3800 2800
-Wire Wire Line
 	3200 2000 3350 2000
 Connection ~ 4000 2000
@@
 $EndComp
 Wire Wire Line
-	4000 2800 4000 2500
-Wire Wire Line
 	4000 2200 4000 2000
 Connection ~ 5050 2000
@@
 Text Label 1950 3500 0    60   ~ 0
 Load
+Wire Wire Line
+	3800 2450 3800 2800
+Wire Wire Line
+	3800 2800 3200 2800
+Wire Wire Line
+	4000 2500 4000 2800
+Wire Wire Line
+	4000 2800 5400 2800
 $EndSCHEMATC
